File: mosfet_v2.kicad_sch (KiCad schematic)
At the start: 26 parts, among them Q10 STL90N6F7, Q11 STL90N6F7, Q12 STL90N6F7, Q7 STL90N6F7, Q8 STL90N6F7, Q9 STL90N6F7

Commit message: reference files added
Parts:
- renumbered C22 to C?, C18 to C?, C21 to C?, C19 to C?, C20 to C?, Q10 to Q?, Q8 to Q?, Q12 to Q?, Q11 to Q?, Q7 to Q?, Q9 to Q?, RGA4 to RGA?, RGA3 to RGA?, RGB6 to RGB?, RGB5 to RGB?, RGB3 to RGB?, RGB4 to RGB?, Rsense_A4 to Rsense_A?, Rsense_A5 to Rsense_A?, Rsense_A6 to Rsense_A?, Rsense_B6 to Rsense_B?, Rsense_B4 to Rsense_B?, Rsense_B5 to Rsense_B?, Rsense_C5 to Rsense_C?, Rsense_C4 to Rsense_C?, Rsense_C6 to Rsense_C?
