File: Ana_ESC.kicad_pcb (KiCad board)
At the start: 4 copper layers, 75 x 75 mm, 99 parts, among them IC3 TCAN330DCNT, J1 BM04B-GHS-TBT_LF__SN__N_, J2 Conn_01x04_Pin, J3 USB_C_Receptacle_USB2.0_16P, J4 BM04B-GHS-TBT_LF__SN__N_, J5 Conn_01x02_Socket, Q10 STL90N6F7, Q11 STL90N6F7, Q12 STL90N6F7, Q7 STL90N6F7, Q8 STL90N6F7, Q9 STL90N6F7, SW1 SW_SPDT, SW2 SW_SPDT, U1 DRV8323RSRGZR, U2 STM32G431CBU6, U3 ME6211C33M5, Y1 ECS-80-20-5PX-TR

Commit message: pcb - mcu part +
Parts:
- added R26: 330R, Resistor_SMD:R_0603_1608Metric_Pad0.98x0.95mm_HandSolder, F.Cu at (58.6, 124.0)
- added R27: 330R, Resistor_SMD:R_0603_1608Metric_Pad0.98x0.95mm_HandSolder, F.Cu at (58.6, 121.0)
- added R28: 330R, Resistor_SMD:R_0603_1608Metric_Pad0.98x0.95mm_HandSolder, F.Cu at (58.6, 118.0)
- moved C18 134.4 mm to (61.5, 98.5)
- moved C19 128.5 mm to (68.5, 90.0)
- moved L3 107.4 mm to (69.5, 118.9), turned to 180 degrees
- moved R25 105.9 mm to (58.5, 100.8), turned to -90 degrees
- moved C42 100.1 mm to (69.6, 115.0)
- moved C43 100.0 mm to (69.6, 116.9)
- moved C24 99.5 mm to (85.7, 81.6)
- moved R23 99.5 mm to (85.8, 79.7)
- moved TH1 99.5 mm to (85.7, 83.5)
- moved C32 95.4 mm to (69.6, 112.9)
- moved C26 94.6 mm to (108.0, 134.5)
- moved R21 84.3 mm to (104.4, 132.9), turned to 180 degrees
- moved R22 83.4 mm to (102.9, 130.9), turned to 180 degrees
- moved D3 34.5 mm to (54.4, 124.0)
- moved D4 30.8 mm to (54.4, 121.0)
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Connections:
- Rsense_A4 pad 1: /Mosfetv2/A- -> GND
- Rsense_A5 pad 1: /Mosfetv2/A- -> GND
- U1 pad 12: /Mosfetv2/A- -> GND
- U2 pad 25: Net-(D3-A) -> Net-(U2-PB12)
- U2 pad 26: Net-(D4-A) -> Net-(U2-PB13)
- U2 pad 27: Net-(D5-A) -> Net-(U2-PB14)
Routing:
- net GND: track 94.2 -> 159.0 mm, vias 24 -> 38
- net /Mosfetv2/A-: track 24.9 -> 0.00 mm, vias 2 -> 0
- net Net-(U2-PF0-OSC_IN): track 0.00 -> 24.0 mm
- net +3.3VA: track 0.00 -> 23.2 mm
- net MCU_PWR: track 1.36 -> 20.8 mm
- net +3.3V: track 5.15 -> 23.0 mm, vias 0 -> 4
- net /MCU/I2C1_SCL: track 0.00 -> 12.3 mm, vias 0 -> 2
- net /MCU/I2C1_SDA: track 0.00 -> 12.1 mm, vias 0 -> 2
- net /MCU/USB_DN: track 3.27 -> 14.4 mm, vias 0 -> 2
- net /MCU/USB_DP: track 3.27 -> 14.0 mm, vias 0 -> 2
- net /MCU/RST: track 3.36 -> 13.6 mm
- net /MCU/NTC_FET: track 3.80 -> 13.3 mm, vias 0 -> 2
- net /Gate_Driver/INLC: track 4.87 -> 13.5 mm, vias 0 -> 1
- net /Gate_Driver/INHC: track 4.48 -> 12.1 mm, vias 0 -> 1
- net /MCU/NTC_MTR: track 7.80 -> 15.3 mm
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Other:
- board size 75 x 75 mm -> 90 x 90 mm

Commit message: all nıght 4/12
Parts:
- added Batt+1: power_pad_smd, Pads:Power_pad_smd, F.Cu at (133.8, 84.5)
- added D6: USBLC6-2SC6Y, LIB_USBLC6-2SC6Y:SOT95P280X145-6N, F.Cu at (63.2, 121.9)
- added GND1: power_pad_smd, Pads:Power_pad_smd, F.Cu at (133.8, 70.8)
- added NT1: NetTie_4, NetTie:NetTie-4_SMD_Pad2.0mm, F.Cu at (113.0, 88.5)
- Q10, Q11, Q12, Q7, Q8, Q9: footprint STL90N6F7:STL90N6F7 -> STL90N6F7:STL90N6F7_Thermal_Vias
- moved C38 94.5 mm to (62.0, 100.5), turned to 90 degrees
- moved C39 93.0 mm to (63.5, 97.5), turned to 180 degrees
- moved C22 92.5 mm to (75.3, 119.0), turned to 180 degrees
- moved C36 85.9 mm to (71.5, 111.0)
- moved U3 84.1 mm to (79.5, 118.2), turned to 180 degrees
- moved C37 84.0 mm to (72.8, 99.5), turned to 90 degrees
- moved C23 74.9 mm to (84.1, 118.3), turned to 180 degrees
- moved D3 42.0 mm to (52.6, 82.0)
- moved D4 42.0 mm to (52.6, 79.0)
- moved D5 42.0 mm to (52.6, 76.0)
- moved R26 42.0 mm to (56.8, 82.0)
- moved R27 42.0 mm to (56.8, 79.0)
- moved R28 42.0 mm to (56.8, 76.0)
- moved R23 41.0 mm to (60.2, 111.8), turned to 180 degrees
- moved C21 39.3 mm to (60.0, 125.3)
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Connections:
- net Net-(IC3-CANH) renamed /MCU/CAN+
- net Net-(IC3-CANL) renamed /MCU/CAN-
- C27 pad 2: GND -> PGND
- C4 pad 2: GND -> /Gate_Driver/PGND
- C5 pad N: GND -> /Gate_Driver/PGND
- J1 pad S1: (no net) -> unconnected-(J1-PadS1)
- J1 pad S2: (no net) -> unconnected-(J1-PadS2)
- J3 pad A6: /MCU/USB_DP -> /MCU/D+
- J3 pad A7: /MCU/USB_DN -> /MCU/D-
- J3 pad B6: /MCU/USB_DP -> /MCU/D+
- J3 pad B7: /MCU/USB_DN -> /MCU/D-
- J4 pad 3: /MCU/I2C1_SDA -> /MCU/I2C1_SCL
- J4 pad S1: (no net) -> unconnected-(J4-PadS1)
- J4 pad S2: (no net) -> unconnected-(J4-PadS2)
- R22 pad 2: /MCU/I2C1_SDA -> /MCU/I2C1_SCL
- Rsense_A4 pad 1: GND -> PGND
- Rsense_A5 pad 1: GND -> PGND
- U1 pad 12: GND -> PGND
- U1 pad 2: GND -> /Gate_Driver/PGND
- U2 pad 45: /MCU/I2C1_SDA -> /MCU/I2C1_SCL
Routing:
- net PGND: track 0.00 -> 24.9 mm, vias 0 -> 42
- net +3.3V: track 23.0 -> 44.7 mm, vias 4 -> 7
- net /Gate_Driver/PGND: track 0.00 -> 15.0 mm, vias 0 -> 6
- net GND: track 159.0 -> 144.2 mm, vias 38 -> 101
- net Net-(U2-PF0-OSC_IN): track 24.0 -> 9.52 mm
- net /MCU/I2C1_SDA: track 12.1 -> 0.00 mm, vias 2 -> 0
- net Net-(IC3-SHDN): track 0.00 -> 10.0 mm, vias 0 -> 2
- net /MCU/I2C1_SCL: track 12.3 -> 21.8 mm, vias 2 -> 4
- net MCU_PWR: track 20.8 -> 30.2 mm, vias 1 -> 2
- net /MCU/CAN+: track 0.00 -> 8.88 mm
- net /MCU/D-: track 0.00 -> 8.37 mm
- net /MCU/D+: track 0.00 -> 8.35 mm
- net VM: track 59.4 -> 51.2 mm, vias 0 -> 7
- net /MCU/CAN-: track 0.00 -> 7.57 mm
- net /MCU/NTC_FET: track 13.3 -> 7.89 mm, vias 2 -> 0
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- added copper zone on B.Cu, net GND
- added copper zone on F.Cu, net PGND

Commit message: all nıght 4/12
Parts:
- moved C16 108.4 mm to (109.5, 112.0)
- moved R10 108.4 mm to (109.5, 110.0)
- moved R9 108.4 mm to (109.5, 108.0)
- moved R8 105.5 mm to (105.1, 115.9)
- moved C15 105.5 mm to (105.1, 118.0)
- moved R7 105.5 mm to (105.1, 113.9)
Routing:
- net /MCU/SWDIO: track 4.78 -> 28.3 mm
- net /MCU/SWCLK: track 3.79 -> 26.3 mm
- net GND: track 144.2 -> 147.6 mm, vias 101 -> 102
- net /Gate_Driver/SHC: vias 54 -> 55
- net /Gate_Driver/SHB: vias 54 -> 55
Changed lines of the file:
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@@
 	(footprint "Capacitor_SMD:C_0603_1608Metric_Pad1.08x0.95mm_HandSolder"
 		(layer "F.Cu")
-		(at 216.0875 92.525 180)
+		(at 109.5 112 180)
 		(descr "Capacitor SMD 0603 (1608 Metric), square (rectangular) end terminal, IPC-7351 nominal with elongated pad for handsoldering. (Body size source: IPC-SM-782 page 76, https://www.pcb-3d.com/wordpress/wp-content/uploads/ipc-sm-782a_amendment_1_and_2.pdf), generated with kicad-footprint-generator")
 		(tags "capacitor handsolder")
@@
 	(footprint "Resistor_SMD:R_0603_1608Metric_Pad0.98x0.95mm_HandSolder"
 		(layer "F.Cu")
-		(at 207.13 88.915)
+		(at 105.13 115.88)
 		(descr "Resistor SMD 0603 (1608 Metric), square (rectangular) end terminal, IPC-7351 nominal with elongated pad for handsoldering. (Body size source: IPC-SM-782 page 72, https://www.pcb-3d.com/wordpress/wp-content/uploads/ipc-sm-782a_amendment_1_and_2.pdf), generated with kicad-footprint-generator")
 		(tags "resistor handsolder")
@@
 	(footprint "Capacitor_SMD:C_0603_1608Metric_Pad1.08x0.95mm_HandSolder"
 		(layer "F.Cu")
-		(at 207.1375 91.035 180)
+		(at 105.1375 118 180)
 		(descr "Capacitor SMD 0603 (1608 Metric), square (rectangular) end terminal, IPC-7351 nominal with elongated pad for handsoldering. (Body size source: IPC-SM-782 page 76, https://www.pcb-3d.com/wordpress/wp-content/uploads/ipc-sm-782a_amendment_1_and_2.pdf), generated with kicad-footprint-generator")
 		(tags "capacitor handsolder")
@@
 	(footprint "Resistor_SMD:R_0603_1608Metric_Pad0.98x0.95mm_HandSolder"
 		(layer "F.Cu")
-		(at 216.0875 88.5)
+		(at 109.5 107.975)
 		(descr "Resistor SMD 0603 (1608 Metric), square (rectangular) end terminal, IPC-7351 nominal with elongated pad for handsoldering. (Body size source: IPC-SM-782 page 72, https://www.pcb-3d.com/wordpress/wp-content/uploads/ipc-sm-782a_amendment_1_and_2.pdf), generated with kicad-footprint-generator")
 		(tags "resistor handsolder")
@@
 	(footprint "Resistor_SMD:R_0603_1608Metric_Pad0.98x0.95mm_HandSolder"
 		(layer "F.Cu")
-		(at 207.1375 86.915)
+		(at 105.1375 113.88)
 		(descr "Resistor SMD 0603 (1608 Metric), square (rectangular) end terminal, IPC-7351 nominal with elongated pad for handsoldering. (Body size source: IPC-SM-782 page 72, https://www.pcb-3d.com/wordpress/wp-content/uploads/ipc-sm-782a_amendment_1_and_2.pdf), generated with kicad-footprint-generator")
 		(tags "resistor handsolder")
@@
 	(footprint "Resistor_SMD:R_0603_1608Metric_Pad0.98x0.95mm_HandSolder"
 		(layer "F.Cu")
-		(at 216.0875 90.525)
+		(at 109.5 110)
 		(descr "Resistor SMD 0603 (1608 Metric), square (rectangular) end terminal, IPC-7351 nominal with elongated pad for handsoldering. (Body size source: IPC-SM-782 page 72, https://www.pcb-3d.com/wordpress/wp-content/uploads/ipc-sm-782a_amendment_1_and_2.pdf), generated with kicad-footprint-generator")
 		(tags "resistor handsolder")
@@
 	)
 	(segment
+		(start 84.9 136.65)
+		(end 84.9 135.9)
+		(width 0.5)
+		(layer "F.Cu")
+		(net 5)
+	)
+	(segment
 		(start 96.5 110.8)
 		(end 96.5 108)
@@
 	)
 	(segment
+		(start 84.9 135.9)
+		(end 83 134)
+		(width 0.5)
+		(layer "F.Cu")
+		(net 5)
+	)
+	(segment
 		(start 71.5175 129.9075)
 		(end 70.25 129.9075)
@@
 	)
 	(segment
-		(start 215.175 90.525)
-		(end 214.0875 90.525)
+		(start 108.5875 110)
+		(end 107.5 110)
 		(width 0.5)
 		(layer "F.Cu")
@@
 	)
 	(segment
-		(start 215.175 90.525)
-		(end 215.175 92.475)
+		(start 108.5875 110)
+		(end 108.5875 111.95)
 		(width 0.5)
 		(layer "F.Cu")
@@
 	)
 	(segment
-		(start 205.0425 90.915)
-		(end 206.155 90.915)
+		(start 103.0425 117.88)
+		(end 104.155 117.88)
 		(width 0.5)
 		(layer "F.Cu")
@@
 	)
 	(segment
-		(start 206.155 90.915)
-		(end 206.275 91.035)
+		(start 104.155 117.88)
+		(end 104.275 118)
 		(width 0.5)
 		(layer "F.Cu")
@@
 	)
 	(segment
-		(start 206.275 88.9725)
-		(end 206.2175 88.915)
+		(start 104.275 115.9375)
+		(end 104.2175 115.88)
 		(width 0.5)
 		(layer "F.Cu")
@@
 	)
 	(segment
-		(start 215.175 92.475)
-		(end 215.225 92.525)
+		(start 108.5875 111.95)
+		(end 108.6375 112)
 		(width 0.5)
 		(layer "F.Cu")
@@
 	)
 	(segment
-		(start 206.275 91.035)
-		(end 206.275 88.9725)
+		(start 104.275 118)
+		(end 104.275 115.9375)
 		(width 0.5)
 		(layer "F.Cu")
@@
 	)
 	(segment
-		(start 214.0875 92.525)
-		(end 215.225 92.525)
+		(start 107.5 112)
+		(end 108.6375 112)
 		(width 0.5)
 		(layer "F.Cu")
@@
 	)
 	(segment
-		(start 205.0425 88.915)
-		(end 206.2175 88.915)
+		(start 103.0425 115.88)
+		(end 104.2175 115.88)
 		(width 0.5)
 		(layer "F.Cu")
@@
 	)
 	(via
-		(at 205.0425 88.915)
+		(at 103.0425 115.88)
 		(size 0.6)
 		(drill 0.3)
@@
 	)
 	(via
+		(at 83 134)
+		(size 0.6)
+		(drill 0.3)
+		(layers "F.Cu" "B.Cu")
+		(net 5)
+	)
+	(via
 		(at 77.25 80.25)
 		(size 0.6)
@@
 	)
 	(via
-		(at 214.0875 90.525)
+		(at 107.5 110)
 		(size 0.6)
 		(drill 0.3)
@@
 	)
 	(via
-		(at 214.0875 92.525)
+		(at 107.5 112)
 		(size 0.6)
 		(drill 0.3)
@@
 	)
 	(via
-		(at 205.0425 90.915)
+		(at 103.0425 117.88)
 		(size 0.6)
 		(drill 0.3)
@@
 	)
 	(segment
-		(start 208 86.965)
-		(end 208.05 86.915)
+		(start 106 113.93)
+		(end 106.05 113.88)
 		(width 0.5)
 		(layer "F.Cu")
@@
 	)
 	(segment
-		(start 208 91.035)
-		(end 208 86.965)
+		(start 106 118)
+		(end 106 113.93)
 		(width 0.5)
 		(layer "F.Cu")
@@
 	)
 	(segment
-		(start 217 90.525)
-		(end 217 92.475)
+		(start 110.4125 110)
+		(end 110.4125 111.95)
 		(width 0.5)
 		(layer "F.Cu")
@@
 	)
 	(segment
-		(start 217 92.475)
-		(end 216.95 92.525)
+		(start 110.4125 111.95)
+		(end 110.3625 112)
 		(width 0.5)
 		(layer "F.Cu")
@@
 	)
 	(segment
-		(start 217 90.525)
-		(end 217 88.5)
+		(start 110.4125 110)
+		(end 110.4125 107.975)
 		(width 0.5)
 		(layer "F.Cu")
@@
 	)
 	(segment
+		(start 52 88)
+		(end 60.5 96.5)
+		(width 0.25)
+		(layer "B.Cu")
+		(net 34)
+	)
+	(segment
+		(start 68.5 96.5)
+		(end 71 99)
+		(width 0.25)
+		(layer "B.Cu")
+		(net 34)
+	)
+	(segment
+		(start 60.5 96.5)
+		(end 68.5 96.5)
+		(width 0.25)
+		(layer "B.Cu")
+		(net 34)
+	)
+	(segment
 		(start 70.25 99.436413)
 		(end 70.137876 99.324289)
@@
 	)
 	(segment
+		(start 68 97)
+		(end 60 97)
+		(width 0.25)
+		(layer "B.Cu")
+		(net 35)
+	)
+	(segment
+		(start 70.137876 99.324289)
+		(end 70.137876 99.137876)
+		(width 0.25)
+		(layer "B.Cu")
+		(net 35)
+	)
+	(segment
+		(start 60 97)
+		(end 52 89)
+		(width 0.25)
+		(layer "B.Cu")
+		(net 35)
+	)
+	(segment
+		(start 70.137876 99.137876)
+		(end 68 97)
+		(width 0.25)
+		(layer "B.Cu")
+		(net 35)
+	)
+	(segment
 		(start 101.9625 130.9)
 		(end 100.375 130.9)
@@
 	(segment
 		(start 92.25 68.7918)
+		(end 92.25 84)
+		(width 0.25)
+		(layer "F.Cu")
+		(net 45)
+	)
+	(segment
+		(start 92.25 84)
 		(end 92.25 90.565)
 		(width 0.25)
@@
 	)
 	(via
+		(at 92.25 84)
+		(size 0.6)
+		(drill 0.3)
+		(layers "F.Cu" "B.Cu")
+		(net 45)
+	)
+	(via
 		(at 98 60)
 		(size 0.6)
@@
 	(segment
 		(start 74.2918 84.5)
-		(end 75.4808 85.689)
+		(end 74.8959 85.1041)
 		(width 0.25)
 		(layer "F.Cu")
@@
 	)
 	(segment
+		(start 74.8959 85.1041)
+		(end 75.4808 85.689)
+		(width 0.25)
+		(layer "F.Cu")
+		(net 49)
+	)
+	(segment
 		(start 74.2918 70)
 		(end 74.2918 84.5)
@@
 		(net 49)
 	)
+	(via
+		(at 74.8959 85.1041)
+		(size 0.6)
+		(drill 0.3)
+		(layers "F.Cu" "B.Cu")
+		(net 49)
+	)
