File: hardware/Ana_ESC2_OneGND_Layer.kicad_pcb (KiCad board)
At the start: 4 copper layers, 90 x 90 mm, 110 parts, among them IC1 TCAN330DCNT, J1 BM04B-GHS-TBT_LF__SN__N_, J2 USB_C_Receptacle_USB2.0_16P, J3 Conn_01x02_Socket, J4 Conn_01x04_Pin, J5 BM04B-GHS-TBT_LF__SN__N_, Q10 STL90N6F7, Q11 STL90N6F7, Q12 STL90N6F7, Q7 STL90N6F7, Q8 STL90N6F7, Q9 STL90N6F7, SW1 SW_SPDT, SW2 SW_SPDT, U1 DRV8323RSRGZR, U2 ME6211C33M5, U3 STM32G431CBU6, Y1 ECS-80-20-5PX-TR

Commit message: final project board layout is in this commit
Parts:
- moved D7 20.3 mm to (102.8, 104.6), turned to 45 degrees
- moved R10 2.01 mm to (108.5, 101.1)
- moved R11 2.01 mm to (108.5, 103.1)
- moved NT1 1.20 mm to (128.5, 77.4)
- renumbered Power_Pad_SMD1 to Batt-1
Connections:
- U3 pad 29: unconnected-(U3-PC6-Pad29) -> /Gate_Driver/CAL
- U3 pad 44: unconnected-(U3-PB6-Pad44) -> /Gate_Driver/FAULT
Routing:
- net (no net): track 26.1 -> 0.00 mm
- net /Gate_Driver/CAL: track 0.00 -> 23.4 mm, vias 0 -> 2
- net /Gate_Driver/FAULT: track 12.2 -> 32.8 mm
- net GND: track 80.1 -> 64.3 mm, vias 69 -> 70
- net MCU_PWR: track 63.9 -> 68.3 mm
- net VM: track 61.0 -> 62.9 mm
- net /Gate_Driver/SHA: track 43.2 -> 44.7 mm, vias 42 -> 43
- net /Gate_Driver/SENS1: track 58.8 -> 60.0 mm
- net /Gate_Driver/SDO: track 35.0 -> 34.4 mm
