File: hardware/Ana_ESC2_OneGND_Layer.kicad_sch (KiCad schematic)
At the start: 4 parts

Commit message: final project board layout is in this commit
Other:
- removed sheet Mosfets
- sheet MCU ports: added CAL, Enable, FAULT; removed NTC_MTR
Changed lines of the file:
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@@
+		)
+	)
+	(wire
+		(pts
+			(xy 82.55 95.25) (xy 114.3 95.25)
+		)
+		(stroke
+			(width 0)
+			(type default)
 		)
 	)
@@
 	(wire
 		(pts
+			(xy 82.55 77.47) (xy 114.3 77.47)
+		)
+		(stroke
+			(width 0)
+			(type default)
+		)
+	)
+	(wire
+		(pts
 			(xy 82.55 111.76) (xy 114.3 111.76)
 		)
@@
 		(pts
 			(xy 166.37 48.26) (xy 189.23 48.26)
+		)
+		(stroke
+			(width 0)
+			(type default)
+		)
+	)
+	(wire
+		(pts
+			(xy 82.55 52.07) (xy 114.3 52.07)
 		)
 		(stroke
@@
 			)
 		)
-		(pin "NTC_MTR" input
-			(at 82.55 95.25 0)
-			(effects
-				(font
-					(size 1.27 1.27)
-				)
-				(justify right)
-			)
-		)
 		(pin "SCLK" output
 			(at 82.55 85.09 0)
@@
 		(pin "SDO" output
 			(at 82.55 90.17 0)
+			(effects
+				(font
+					(size 1.27 1.27)
+				)
+				(justify right)
+			)
+		)
+		(pin "CAL" output
+			(at 82.55 77.47 0)
+			(effects
+				(font
+					(size 1.27 1.27)
+				)
+				(justify right)
+			)
+		)
+		(pin "FAULT" input
+			(at 82.55 95.25 0)
+			(effects
+				(font
+					(size 1.27 1.27)
+				)
+				(justify right)
+			)
+		)
+		(pin "Enable" output
+			(at 82.55 52.07 0)
 			(effects
 				(font
@@
 				(path "/57129761-6d47-486c-bd7a-90dbb6f75754"
 					(page "4")
-				)
-			)
-		)
-	)
-	(sheet
-		(at 49.53 124.46)
-		(size 43.18 69.85)
-		(exclude_from_sim yes)
-		(in_bom no)
-		(on_board no)
-		(dnp yes)
-		(fields_autoplaced yes)
-		(stroke
-			(width 0.1524)
-			(type solid)
-		)
-		(fill
-			(color 0 0 0 0.0000)
-		)
-		(property "Sheetname" "Mosfets"
-			(at 49.53 123.7484 0)
-			(effects
-				(font
-					(size 1.27 1.27)
-				)
-				(justify left bottom)
-			)
-		)
-		(property "Sheetfile" "Mosfets.kicad_sch"
-			(at 49.53 194.8946 0)
-			(effects
-				(font
-					(size 1.27 1.27)
-				)
-				(justify left top)
-			)
-		)
-		(pin "FAZ_A" output
-			(at 92.71 134.62 0)
-			(effects
-				(font
-					(size 1.27 1.27)
-				)
-				(justify right)
-			)
-		)
-		(pin "FAZ_B" output
-			(at 92.71 139.7 0)
-			(effects
-				(font
-					(size 1.27 1.27)
-				)
-				(justify right)
-			)
-		)
-		(pin "FAZ_C" output
-			(at 92.71 144.78 0)
-			(effects
-				(font
-					(size 1.27 1.27)
-				)
-				(justify right)
-			)
-		)
-		(pin "GHA" input
-			(at 49.53 129.54 180)
-			(effects
-				(font
-					(size 1.27 1.27)
-				)
-				(justify left)
-			)
-		)
-		(pin "GHB" input
-			(at 49.53 132.08 180)
-			(effects
-				(font
-					(size 1.27 1.27)
-				)
-				(justify left)
-			)
-		)
-		(pin "GHC" input
-			(at 49.53 134.62 180)
-			(effects
-				(font
-					(size 1.27 1.27)
-				)
-				(justify left)
-			)
-		)
-		(pin "GLA" input
-			(at 49.53 138.43 180)
-			(effects
-				(font
-					(size 1.27 1.27)
-				)
-				(justify left)
-			)
-		)
-		(pin "GLB" input
-			(at 49.53 140.97 180)
-			(effects
-				(font
-					(size 1.27 1.27)
-				)
-				(justify left)
-			)
-		)
-		(pin "GLC" input
-			(at 49.53 143.51 180)
-			(effects
-				(font
-					(size 1.27 1.27)
-				)
-				(justify left)
-			)
-		)
-		(pin "SHA" output
-			(at 49.53 158.75 180)
-			(effects
-				(font
-					(size 1.27 1.27)
-				)
-				(justify left)
-			)
-		)
-		(pin "SHB" output
-			(at 49.53 161.29 180)
-			(effects
-				(font
-					(size 1.27 1.27)
-				)
-				(justify left)
-			)
-		)
-		(pin "SHC" output
-			(at 49.53 163.83 180)
-			(effects
-				(font
-					(size 1.27 1.27)
-				)
-				(justify left)
-			)
-		)
-		(pin "SNA" output
-			(at 49.53 170.18 180)
-			(effects
-				(font
-					(size 1.27 1.27)
-				)
-				(justify left)
-			)
-		)
-		(pin "SNB" output
-			(at 49.53 172.72 180)
-			(effects
-				(font
-					(size 1.27 1.27)
-				)
-				(justify left)
-			)
-		)
-		(pin "SNC" output
-			(at 49.53 175.26 180)
-			(effects
-				(font
-					(size 1.27 1.27)
-				)
-				(justify left)
-			)
-		)
-		(pin "SPA" output
-			(at 49.53 179.07 180)
-			(effects
-				(font
-					(size 1.27 1.27)
-				)
-				(justify left)
-			)
-		)
-		(pin "SPB" output
-			(at 49.53 181.61 180)
-			(effects
-				(font
-					(size 1.27 1.27)
-				)
-				(justify left)
-			)
-		)
-		(pin "SPC" output
-			(at 49.53 184.15 180)
-			(effects
-				(font
-					(size 1.27 1.27)
-				)
-				(justify left)
-			)
-		)
-		(pin "Vdrain" output
-			(at 49.53 125.73 180)
-			(effects
-				(font
-					(size 1.27 1.27)
-				)
-				(justify left)
-			)
-		)
-		(instances
-			(project "Ana_ESC2_OneGND_Layer"
-				(path "/57129761-6d47-486c-bd7a-90dbb6f75754"
-					(page "2")
 				)
 			)
@@
 			)
 		)
-		(pin "FAULT" input
+		(pin "FAULT" output
 			(at 114.3 95.25 180)
 			(effects
