File: hardware/Ana_ESC2_OneGND_Layer.kicad_sch (KiCad schematic)
At the start: 4 parts

Commit message: After graduation presantition. USB differantial ways improved for usb connection issue. DRV83233 Enable and nSCS pins changed to be in true connection with STM32G431. ETC
Other:
- sheet Gate_Driver ports: added nSCS; removed none
- sheet MCU ports: added nSCS; removed none
Changed lines of the file:
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@@
+	(wire
+		(pts
+			(xy 82.55 48.26) (xy 114.3 48.26)
+		)
+		(stroke
+			(width 0)
+			(type default)
+		)
+	)
 	(wire
 		(pts
@@
 			)
 		)
+		(pin "nSCS" output
+			(at 82.55 48.26 0)
+			(effects
+				(font
+					(size 1.27 1.27)
+				)
+				(justify right)
+			)
+		)
 		(instances
 			(project "Ana_ESC2_OneGND_Layer"
@@
 			(effects
 				(font
+					(size 1.27 1.27)
+				)
+				(justify left)
+			)
+		)
+		(pin "nSCS" input
+			(at 114.3 48.26 180)
+			(effects
+				(font
