File: hardware/MCU.kicad_sch (KiCad schematic)
At the start: 48 parts, among them IC1 TCAN330DCNT, J1 BM04B-GHS-TBT_LF__SN__N_, J2 USB_C_Receptacle_USB2.0_16P, J3 Conn_01x02_Socket, J4 Conn_01x04_Pin, J5 BM04B-GHS-TBT_LF__SN__N_, SW2 SW_SPDT, U2 ME6211C33M5, U3 STM32G431CBU6, Y1 ECS-80-20-5PX-TR

Commit message: After graduation presantition. USB differantial ways improved for usb connection issue. DRV83233 Enable and nSCS pins changed to be in true connection with STM32G431. ETC
Parts:
- added R1, R2: 5.1k, Resistor_SMD:R_0603_1608Metric_Pad0.98x0.95mm_HandSolder, symbol Device:R_Small
- renumbered w to w1
Connections:
- net GND2: now also R1.1, R2.1
- net VBus: now also R23.1, R24.2
- net nSCS: now reaches U3.22 (PB10)
- net at J2.A5 (CC1): now also R1.2
- net at J2.B5 (CC2): now also R2.2
- no-connect marks 17 -> 14
Other:
- moved on the sheet: C32
