File: hardware/mosfetv2.kicad_sch (KiCad schematic)
At the start: 26 parts, among them Q10 STL90N6F7, Q11 STL90N6F7, Q12 STL90N6F7, Q7 STL90N6F7, Q8 STL90N6F7, Q9 STL90N6F7

Commit message: final project board layout is in this commit
Parts:
- renumbered Power_Pad_SMD1 to Batt-1
Other:
- note added: "I = 15A RDSON = 0.005 OHM PLOSS = I^2 * R PLOSS = 1.125 W ----- RDSON(T=125) = 1.5*0.005 = 0.0075 OHM PLOSS = 1.6875 W ----- MOSFET TEMPERATURE = 25 + 1.6875 * 31.3 = 77.81 C"
Changed lines of the file:
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@@
 		)
 	)
+	(text "I = 15A\nRDSON = 0.005 OHM\nPLOSS = I^2 * R\nPLOSS = 1.125 W\n-----\nRDSON(T=125) = 1.5*0.005 = 0.0075 OHM\nPLOSS = 1.6875 W\n-----\nMOSFET TEMPERATURE\n= 25 + 1.6875 * 31.3\n= 77.81 C\n"
+		(exclude_from_sim no)
+		(at 55.372 390.652 0)
+		(effects
+			(font
+				(size 1.27 1.27)
+			)
+			(justify left)
+		)
+	)
 	(text "Bu değeri biraza daha düşürebiliriz thermal vialar ile"
 		(exclude_from_sim no)
@@
 		(dnp no)
 		(fields_autoplaced yes)
-		(property "Reference" "Power_Pad_SMD1"
+		(property "Reference" "Batt-1"
 			(at 62.23 31.7499 0)
 			(effects
@@
 			(project ""
 				(path "/57129761-6d47-486c-bd7a-90dbb6f75754/a2e9c01f-dc3c-42e3-9ad2-b4c7bc962bba"
-					(reference "Power_Pad_SMD1")
+					(reference "Batt-1")
 					(unit 1)
 				)
